File: Projekt_EAGLE/0.1.brd (EAGLE design)
At the start: 289.2 x 129.4 mm, 320 parts, among them IC1 TCA9548A, P1 53048-0210, P2 53048-0410, P3 53048-0410, P4 53048-0410, Q1 16MHz, Q2 32.768kHz, T1 SOT89 NPN BCE, T2 SOT89 NPN BCE, T3 SOT89 NPN BCE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

Commit message: Uaktualniony schemat EAGLE.
Parts:
- removed X5: 52745-3090, con-molex:52745-3090
- added JP4: (no value), pinhead:1X02
- added SJ6, SJ7, SJ8: (no value), jumper:SJ_2
- added X6: FH12-30S-0.5SH, con-hirose:FH12-30S-0.5SH
- JP2: device pinhead:1X04 -> pinhead:1X02
- moved JP2 48.8 mm to (293.4, 139.1), turned to 180 degrees
- moved C10 7.99 mm to (253.0, 107.3), turned to 90 degrees
- moved R70 1.91 mm to (295.9, 92.8)
- moved C45 0.63 mm to (299.0, 91.5)
Connections:
- removed net I2C_2_SCL: U3.29
- removed net I2C_2_SDA: U3.30
- removed net UART_EXT_RX: JP2.3, U3.52
- removed net UART_EXT_TX: JP2.2, U3.51
- new net BOOT0: SJ6.2, U3.60
- new net BOOT1: SJ7.2, U3.28
- new net EXT_RX: JP4.1, U3.43
- new net EXT_TX: JP4.2, U3.42
- new net N$77: L1.2, SJ8.2
- new net OLED_BIG_CS: U3.51, X6.14
- net +3V3: now also SJ6.3, SJ7.3, SJ8.3; no longer JP2.1
- net +5V: now also JP2.1, SJ8.1; no longer L1.2
- net GND: now also JP2.2, SJ6.1, SJ7.1, X6.11, X6.12, X6.17, X6.18, X6.2; no longer JP2.4, U3.60, X5.11, X5.12, X5.14, X5.17, X5.18, X5.2
- net IREF: now also X6.27; no longer X5.27
- net MCU_2_RX: now also U3.29; no longer U3.42
- net MCU_2_TX: now also U3.30; no longer U3.43
- net N$24: now also X6.29; no longer X5.29
- net OLED_BIG_CLK: now also X6.19; no longer X5.19
- net OLED_BIG_DC: now also X6.16; no longer X5.16
- net OLED_BIG_MOSI: now also X6.20; no longer X5.20
- net OLED_BIG_RES: now also X6.15; no longer X5.15
- net VCOMH: now also X6.28; no longer X5.28
- net VDD: now also X6.10; no longer X5.10
Routing:
- net OLED_BIG_CS: track 0.00 -> 52.0 mm, vias 0 -> 1
- net BOOT0: track 0.00 -> 27.2 mm, vias 0 -> 2
- net UART_EXT_RX: track 24.7 -> 0.00 mm
- net +3V3: track 1203.8 -> 1228.4 mm, vias 16 -> 19
- net MCU_2_TX: track 90.3 -> 69.0 mm
- net UART_EXT_TX: track 20.7 -> 0.00 mm
- net MCU_2_RX: track 82.8 -> 62.4 mm
- net BOOT1: track 0.00 -> 20.0 mm, vias 0 -> 2
- net GND: track 2804.5 -> 2784.8 mm
- net EXT_TX: track 0.00 -> 17.9 mm
- net EXT_RX: track 0.00 -> 16.2 mm
- net N$61: track 95.9 -> 102.8 mm, vias 6 -> 7
- net N$77: track 0.00 -> 4.73 mm
- net CAN_RXD: track 264.2 -> 267.7 mm
- net I2C_RESET: track 37.2 -> 34.1 mm
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Other:
- board text added: "10.03.2020"
- board text added: "designed by Marcin Szykowny for PUT Solar Dynamics 2020"
- board text added: "v. 2.3"
- board text removed: "26.11.2018"
- board text removed: "3V3"
- board text removed: "EXT UART"
- board text removed: "designed by Marcin Szykowny for PUT Solar Dynamics 2018"
- board text removed: "v. 2.1"
