File: Projekt_EAGLE/0.1.sch (EAGLE design)
At the start: 320 parts, among them IC1 TCA9548A, P1 53048-0210, P2 53048-0410, P3 53048-0410, P4 53048-0410, Q1 16MHz, Q2 32.768kHz, T1 SOT89 NPN BCE, T2 SOT89 NPN BCE, T3 SOT89 NPN BCE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

Commit message: Uaktualniony schemat EAGLE.
Parts:
- removed X5: 52745-3090, con-molex:52745-3090
- added JP4: (no value), pinhead:PINHD-1X2
- added SJ6, SJ7, SJ8: (no value), jumper:SJ2W
- added X6: FH12-30S-0.5SH, con-hirose:FH12-30S-0.5SH
- JP2: device pinhead:PINHD-1X4 -> pinhead:PINHD-1X2
Connections:
- removed net I2C_2_SCL: U3.PB10
- removed net I2C_2_SDA: U3.PB11
- removed net UART_EXT_RX: JP2.3, U3.PC11
- removed net UART_EXT_TX: JP2.2, U3.PC10
- new net BOOT0: SJ6.2, U3.BOOT0
- new net BOOT1: SJ7.2, U3.PB1_2
- new net EXT_RX: JP4.1, U3.PA10
- new net EXT_TX: JP4.2, U3.PA9
- new net N$77: L1.2, SJ8.2
- new net OLED_BIG_CS: U3.PC10, X6-14.1
- net +3V3: now also SJ6.3, SJ7.3, SJ8.3; no longer JP2.1
- net +5V: now also JP2.1, SJ8.1; no longer L1.2
- net GND: now also JP2.2, SJ6.1, SJ7.1, X6-11.1, X6-12.1, X6-17.1, X6-18.1, X6-2.1; no longer JP2.4, U3.BOOT0, X5-11.S, X5-12.S, X5-14.S, X5-17.S, X5-18.S, X5-2.S
- net IREF: now also X6-27.1; no longer X5-27.S
- net MCU_2_RX: now also U3.PB10; no longer U3.PA9
- net MCU_2_TX: now also U3.PB11; no longer U3.PA10
- net N$24: now also X6-29.1; no longer X5-29.S
- net OLED_BIG_CLK: now also X6-19.1; no longer X5-19.S
- net OLED_BIG_DC: now also X6-16.1; no longer X5-16.S
- net OLED_BIG_MOSI: now also X6-20.1; no longer X5-20.S
- net OLED_BIG_RES: now also X6-15.1; no longer X5-15.S
- net VCOMH: now also X6-28.1; no longer X5-28.S
- net VDD: now also X6-10.1; no longer X5-10.S
Other:
- note removed: "BS1"
- note removed: "BS2"
- note removed: "CS#"
- note removed: "D/C#"
- note removed: "D0"
- note removed: "D1"
- note removed: "D2"
- note removed: "D3"
- note removed: "D4"
- note removed: "D5"
- note removed: "D6"
- note removed: "D7"
- note removed: "E/RD#"
- note removed: "IREF"
- note removed: "NC"
- note removed: "R/W#"
- note removed: "RES#"
- note removed: "VCC"
- note removed: "VCOMH"
- note removed: "VDD"
- note removed: "VSS"
